File: hardware/ap206-pll.sch (KiCad schematic (older format))
At the start: 35 parts, among them CON1 AVR-ISP-6, J1 Screw_Terminal_01x06, J2 Screw_Terminal_01x05, SW1 QLOCK, U1 4069, U2 LM7805_TO220, U4 ATTINY25-20PU, U6 4504, U7 4046, Y1 11.0592

Commit message: Initial tested and working version, with fixes
Parts:
- J1: Part# (none) -> 1985001
- J2: Part# (none) -> 1989777
- SW1: footprint Button_Switch_THT:SW_E-Switch_EG1271_DPDT -> Button_Switch_THT:SW_CuK_JS202011CQN_DPDT_Straight
Connections:
- net 12(WHTBLK): now also J2.1 (Pin_1), SW1.3 (C); no longer J2.2 (Pin_2), SW1.2 (B)
- net 13(GRY): now also J2.2 (Pin_2), SW1.2 (B); no longer J2.1 (Pin_1), SW1.3 (C)
Changed lines of the file:
@@
 F 2 "TerminalBlock_Phoenix:TerminalBlock_Phoenix_PT-1,5-6-3.5-H_1x06_P3.50mm_Horizontal" H 600 1400 50  0001 C CNN
 F 3 "~" H 600 1400 50  0001 C CNN
+F 4 "1985001" H 600 1400 50  0001 C CNN "Part#"
 	1    600  1400
 	-1   0    0    -1
@@
 F 0 "SW1" H 9400 1335 50  0000 C CNN
 F 1 "QLOCK" H 9400 1244 50  0000 C CNN
-F 2 "Button_Switch_THT:SW_E-Switch_EG1271_DPDT" H 9400 1050 50  0001 C CNN
+F 2 "Button_Switch_THT:SW_CuK_JS202011CQN_DPDT_Straight" H 9400 1050 50  0001 C CNN
 F 3 "" H 9400 1050 50  0001 C CNN
 	1    9400 1050
@@
 F 2 "TerminalBlock_Phoenix:TerminalBlock_Phoenix_PT-1,5-5-3.5-H_1x05_P3.50mm_Horizontal" H 8300 1250 50  0001 C CNN
 F 3 "~" H 8300 1250 50  0001 C CNN
+F 4 "1989777" H 8300 1250 50  0001 C CNN "Part#"
 	1    8300 1250
 	-1   0    0    -1
 $EndComp
-Text Label 8700 1050 0    50   ~ 0
+Text Label 8700 1150 0    50   ~ 0
 13(GRY)
 Wire Wire Line
@@
 F 0 "SW1" H 9400 1835 50  0000 C CNN
 F 1 "QLOCK" H 9400 1744 50  0000 C CNN
-F 2 "Button_Switch_THT:SW_E-Switch_EG1271_DPDT" H 9400 1550 50  0001 C CNN
+F 2 "Button_Switch_THT:SW_CuK_JS202011CQN_DPDT_Straight" H 9400 1550 50  0001 C CNN
 F 3 "" H 9400 1550 50  0001 C CNN
 	2    9400 1550
 	1    0    0    -1
 $EndComp
-Text Label 8700 1150 0    50   ~ 0
+Text Label 8700 1050 0    50   ~ 0
 12(WHTBLK)
 Wire Wire Line

Commit message: Add documentation and symbol cache (for CADLAB)
Connections:
- net 19(WHT) renamed 9(WHT)
Changed lines of the file:
@@
 	8500 1450 9100 1450
 Text Label 8700 1450 0    50   ~ 0
-19(WHT)
+9(WHT)
 Wire Wire Line
 	9600 1450 9700 1450
